File: Duck.kicad_sch (KiCad schematic)
At the start: 32 parts, among them J1 Conn_01x02, J2 USB_C_Receptacle_USB2.0_14P, SW1 SW_Push, U1 RP2040, U2 MAX98357A, U3 W25Q128JVS, U4 MCP1700x-120xxMB, Y1 Crystal_GND24

Commit message: All of the pcb stuff
I kinda forgot to comit lol
Parts:
- removed J2: USB_C_Receptacle_USB2.0_14P, symbol Connector:USB_C_Receptacle_USB2.0_14P
- removed R3, R4: 5.1k, symbol Device:R
- removed U4: MCP1700x-120xxMB, Package_TO_SOT_SMD:SOT-89-3, symbol Regulator_Linear:MCP1700x-120xxMB
- added C18: 0.1uF, Capacitor_SMD:C_0402_1005Metric, symbol Device:C
- added C19, C20: 10uF, Capacitor_SMD:C_0201_0603Metric, symbol Device:C
- added C21: 10uf, Capacitor_SMD:C_0201_0603Metric, symbol Device:C
- added D1: SK6812MINI-E, LED_SMD:LED_SK6812MINI-E_3.2x2.8mm_P1.5mm_ReverseMount, symbol LED:SK6812MINI-E
- added D3: D, Diode_SMD:D_0402_1005Metric, symbol Device:D
- added J3: Conn_02x01, Connector_PinSocket_2.54mm:PinSocket_1x02_P2.54mm_Vertical, symbol Connector_Generic:Conn_02x01
- added R10: 330, Resistor_SMD:R_0402_1005Metric, symbol Device:R
- added R11: 2k, Resistor_SMD:R_0402_1005Metric, symbol Device:R
- added R12, R13: 5.1k, Resistor_SMD:R_0402_1005Metric, symbol Device:R
- added R8: 100k, Resistor_SMD:R_0402_1005Metric, symbol Device:R
- added R9: 1000k, Resistor_SMD:R_0402_1005Metric, symbol Device:R
- added SW2: SW_Push, MX_Alps_Hybrid:MX-1.5U, symbol Switch:SW_Push
- added U4: MCP73831-2-OT, Package_TO_SOT_SMD:SOT-23-5, symbol Battery_Management:MCP73831-2-OT
- added U5: NCP1117-3.3_SOT223, Package_TO_SOT_SMD:SOT-223-3_TabPin2, symbol Regulator_Linear:NCP1117-3.3_SOT223
- added USBC1: TYPE-C-31-M-12, easyeda2kicad:USB-C_SMD-TYPE-C-31-M-12_1, symbol easyeda2kicad:TYPE-C-31-M-12
- C1, C10, C11, C12, C17, C2, C3, C4, C5, C6, C7, C8, C9: footprint (none) -> Capacitor_SMD:C_0402_1005Metric
- C13, C14: footprint (none) -> Capacitor_SMD:C_0603_1608Metric
- C15, C16: value 15pF -> 33pF; footprint (none) -> Capacitor_SMD:C_0402_1005Metric
- J1: footprint (none) -> Connector_PinSocket_2.54mm:PinSocket_1x02_P2.54mm_Vertical
- R1, R2, R5, R6, R7: footprint (none) -> Resistor_SMD:R_0402_1005Metric
- SW1: footprint (none) -> easyeda2kicad:SW-SMD_L3.9-W3.0-P4.45
- Y1: footprint (none) -> easyeda2kicad:CRYSTAL-SMD_4P-L3.2-W2.5-BL
Connections:
- net +3.3V: now also C14.1, U1.26 (RUN), C18.2, C19.2, U5.2 (VO)
- net GND: now also U1.19 (TESTEN), U2.17 (PAD), U2.2 (GAIN_SLOT), C18.1, C19.1, C20.2, C21.2, D1.1 (VSS), R11.1, R12.1, R13.2, R9.2, SW2.2, U4.2 (V_{SS}), U5.1 (GND), USBC1.B1A12 (GND)
- net USB_D+: now also R2.1, USBC1.A6 (DP1), USBC1.B6 (DP2); no longer R1.1
- net USB_D-: now also R1.1, USBC1.A7 (DN1), USBC1.B7 (DN2); no longer R2.1
- net VBUS: now also C21.1, D3.1 (K), U4.4 (V_{DD}), U5.3 (VI), USBC1.A4B9 (VBUS)
- net MAXSLEEP: now reaches U1.14 (GPIO11)
- net MAXSLEEP: now also R8.2
- net NEOPIXEL INPUT: now reaches U1.5 (GPIO3)
- net NEOPIXEL INPUT: now also R10.1
- net at U1.6 (GPIO4): now also SW2.1
- net at U2.4 (~{SD_MODE}): now also R8.1
- new net: R12.2, USBC1.A5 (CC1)
- new net: R11.2, U4.5 (PROG)
- new net: D1.2 (DIN), R10.2
- new net: R9.1, USBC1.1 (EH), USBC1.2 (EH), USBC1.3 (EH), USBC1.4 (EH)
- new net: R13.1, USBC1.B5 (CC2)
- new net VBAT: C20.1, D3.2 (A), J3.1 (Pin_1), J3.2 (Pin_2), U4.3 (V_{BAT})
- new net VDD: D1.3 (VDD)
- no-connect marks 0 -> 28
Other:
- moved on the sheet: C1, C10, C11, C12, C13, C14, C15, C16, C17, C2, C3, C4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
